Commit message: fix(jettank): optimize tracked tank skid-steer kinematics and align with paper benchmark

File: 04_demo_simulation/ros1/mars_online_jettank/urdf/jettank.urdf.xacro (robot description, xacro)
@@ -123,5 +123,5 @@
   </link>
   <joint name="laser_joint" type="fixed">
-    <origin xyz="0.05 0 0.11" rpy="0 0 0"/>
+    <origin xyz="0 0 0.11" rpy="0 0 0"/>
     <parent link="base_link"/>
     <child link="laser_frame"/>

Commit message: feat(jettank): add realistic caterpillar tank tracks model and eliminate self-chassis clearance stall

File: 04_demo_simulation/ros1/mars_online_jettank/urdf/jettank.urdf.xacro (robot description, xacro)
@@ -41,24 +41,76 @@
     </visual>
   </link>
-  <!-- Left Track / Wheel -->
+  <!-- Left Caterpillar Track Assembly (Dải bánh xích xe tăng bên trái) -->
   <link name="left_wheel">
     <inertial>
-      <mass value="0.4"/>
-      <origin xyz="0 0 0" rpy="1.5707963 0 0"/>
-      <inertia ixx="0.0006" ixy="0" ixz="0" iyy="0.0006" iyz="0" izz="0.0008"/>
+      <mass value="0.8"/>
+      <origin xyz="0 0 0" rpy="0 0 0"/>
+      <inertia ixx="0.001" ixy="0" ixz="0" iyy="0.003" iyz="0" izz="0.003"/>
     </inertial>
+    <!-- Collision: main driving track base for skid-steer friction -->
     <collision>
       <origin xyz="0 0 0" rpy="1.5707963 0 0"/>
       <geometry>
-        <cylinder radius="0.045" length="0.04"/>
+        <cylinder radius="0.045" length="0.045"/>
       </geometry>
     </collision>
-    <visual>
-      <origin xyz="0 0 0" rpy="1.5707963 0 0"/>
-      <geometry>
-        <cylinder radius="0.045" length="0.04"/>
-      </geometry>
-      <material name="black">
+    <!-- Visual 1: Main continuous black rubber caterpillar track belt -->
+    <visual>
+      <origin xyz="0 0 0" rpy="0 0 0"/>
+      <geometry>
+        <box size="0.25 0.045 0.07"/>
+      </geometry>
+      <material name="track_rubber">
         <color rgba="0.1 0.1 0.1 1.0"/>
+      </material>
+    </visual>
+    <!-- Visual 2: Front driving sprocket wheel -->
+    <visual>
+      <origin xyz="0.095 0 0" rpy="1.5707963 0 0"/>
+      <geometry>
+        <cylinder radius="0.035" length="0.047"/>
+      </geometry>
+      <material name="track_wheel">
+        <color rgba="0.25 0.28 0.32 1.0"/>
+      </material>
+    </visual>
+    <!-- Visual 3: Rear idler sprocket wheel -->
+    <visual>
+      <origin xyz="-0.095 0 0" rpy="1.5707963 0 0"/>
+      <geometry>
+        <cylinder radius="0.035" length="0.047"/>
+      </geometry>
+      <material name="track_wheel">
+        <color rgba="0.25 0.28 0.32 1.0"/>
+      </material>
+    </visual>
+    <!-- Visual 4: Middle road wheel 1 -->
+    <visual>
+      <origin xyz="-0.032 0 -0.005" rpy="1.5707963 0 0"/>
+      <geometry>
+        <cylinder radius="0.030" length="0.047"/>
+      </geometry>
+      <material name="track_wheel">
+        <color rgba="0.35 0.38 0.42 1.0"/>
+      </material>
+    </visual>
+    <!-- Visual 5: Middle road wheel 2 -->
+    <visual>
+      <origin xyz="0.032 0 -0.005" rpy="1.5707963 0 0"/>
+      <geometry>
+        <cylinder radius="0.030" length="0.047"/>
+      </geometry>
+      <material name="track_wheel">
+        <color rgba="0.35 0.38 0.42 1.0"/>
+      </material>
+    </visual>
+    <!-- Visual 6: Track top mudguard / fender -->
+    <visual>
+      <origin xyz="0 0 0.04" rpy="0 0 0"/>
+      <geometry>
+        <box size="0.26 0.05 0.008"/>
+      </geometry>
+      <material name="dark_gray">
+        <color rgba="0.2 0.22 0.25 1.0"/>
       </material>
     </visual>
@@ -70,24 +122,76 @@
     <axis xyz="0 1 0"/>
   </joint>
-  <!-- Right Track / Wheel -->
+  <!-- Right Caterpillar Track Assembly (Dải bánh xích xe tăng bên phải) -->
   <link name="right_wheel">
     <inertial>
-      <mass value="0.4"/>
-      <origin xyz="0 0 0" rpy="1.5707963 0 0"/>
-      <inertia ixx="0.0006" ixy="0" ixz="0" iyy="0.0006" iyz="0" izz="0.0008"/>
+      <mass value="0.8"/>
+      <origin xyz="0 0 0" rpy="0 0 0"/>
+      <inertia ixx="0.001" ixy="0" ixz="0" iyy="0.003" iyz="0" izz="0.003"/>
     </inertial>
+    <!-- Collision: main driving track base for skid-steer friction -->
     <collision>
       <origin xyz="0 0 0" rpy="1.5707963 0 0"/>
       <geometry>
-        <cylinder radius="0.045" length="0.04"/>
+        <cylinder radius="0.045" length="0.045"/>
       </geometry>
     </collision>
-    <visual>
-      <origin xyz="0 0 0" rpy="1.5707963 0 0"/>
-      <geometry>
-        <cylinder radius="0.045" length="0.04"/>
-      </geometry>
-      <material name="black">
+    <!-- Visual 1: Main continuous black rubber caterpillar track belt -->
+    <visual>
+      <origin xyz="0 0 0" rpy="0 0 0"/>
+      <geometry>
+        <box size="0.25 0.045 0.07"/>
+      </geometry>
+      <material name="track_rubber">
         <color rgba="0.1 0.1 0.1 1.0"/>
+      </material>
+    </visual>
+    <!-- Visual 2: Front driving sprocket wheel -->
+    <visual>
+      <origin xyz="0.095 0 0" rpy="1.5707963 0 0"/>
+      <geometry>
+        <cylinder radius="0.035" length="0.047"/>
+      </geometry>
+      <material name="track_wheel">
+        <color rgba="0.25 0.28 0.32 1.0"/>
+      </material>
+    </visual>
+    <!-- Visual 3: Rear idler sprocket wheel -->
+    <visual>
+      <origin xyz="-0.095 0 0" rpy="1.5707963 0 0"/>
+      <geometry>
+        <cylinder radius="0.035" length="0.047"/>
+      </geometry>
+      <material name="track_wheel">
+        <color rgba="0.25 0.28 0.32 1.0"/>
+      </material>
+    </visual>
+    <!-- Visual 4: Middle road wheel 1 -->
+    <visual>
+      <origin xyz="-0.032 0 -0.005" rpy="1.5707963 0 0"/>
+      <geometry>
+        <cylinder radius="0.030" length="0.047"/>
+      </geometry>
+      <material name="track_wheel">
+        <color rgba="0.35 0.38 0.42 1.0"/>
+      </material>
+    </visual>
+    <!-- Visual 5: Middle road wheel 2 -->
+    <visual>
+      <origin xyz="0.032 0 -0.005" rpy="1.5707963 0 0"/>
+      <geometry>
+        <cylinder radius="0.030" length="0.047"/>
+      </geometry>
+      <material name="track_wheel">
+        <color rgba="0.35 0.38 0.42 1.0"/>
+      </material>
+    </visual>
+    <!-- Visual 6: Track top mudguard / fender -->
+    <visual>
+      <origin xyz="0 0 0.04" rpy="0 0 0"/>
+      <geometry>
+        <box size="0.26 0.05 0.008"/>
+      </geometry>
+      <material name="dark_gray">
+        <color rgba="0.2 0.22 0.25 1.0"/>
       </material>
     </visual>
@@ -99,5 +203,5 @@
     <axis xyz="0 1 0"/>
   </joint>
-  <!-- Lidar mount & sensor -->
+  <!-- Lidar mount mast & sensor (elevated above chassis for clean 360-degree view) -->
   <link name="laser_frame">
     <inertial>
@@ -121,7 +225,17 @@
       </material>
     </visual>
+    <!-- Visual mast / support bracket -->
+    <visual>
+      <origin xyz="0 0 -0.035" rpy="0 0 0"/>
+      <geometry>
+        <cylinder radius="0.015" length="0.07"/>
+      </geometry>
+      <material name="dark_gray">
+        <color rgba="0.2 0.22 0.25 1.0"/>
+      </material>
+    </visual>
   </link>
   <joint name="laser_joint" type="fixed">
-    <origin xyz="0 0 0.11" rpy="0 0 0"/>
+    <origin xyz="0 0 0.16" rpy="0 0 0"/>
     <parent link="base_link"/>
     <child link="laser_frame"/>
@@ -194,5 +308,5 @@
         </scan>
         <range>
-          <min>0.10</min>
+          <min>0.15</min>
           <max>1.60</max>
           <resolution>0.01</resolution>

Commit message: feat(robot-model): redesign JetTank tracked chassis matching Hiwonder photo & set pure red entry and pure blue return paths

File: 04_demo_simulation/ros1/mars_online_jettank/urdf/jettank.urdf.xacro (robot description, xacro)
@@ -1,4 +1,20 @@
 <?xml version="1.0"?>
 <robot name="jettank" xmlns:xacro="http://ros.org/wiki/xacro">
+  <!-- Materials matching official Hiwonder JetTank metallic green & matte black hardware -->
+  <material name="hiwonder_green">
+    <color rgba="0.13 0.69 0.35 1.0"/>
+  </material>
+  <material name="jet_black">
+    <color rgba="0.12 0.12 0.14 1.0"/>
+  </material>
+  <material name="matte_track">
+    <color rgba="0.18 0.18 0.20 1.0"/>
+  </material>
+  <material name="metal_silver">
+    <color rgba="0.75 0.78 0.82 1.0"/>
+  </material>
+  <material name="lens_glass">
+    <color rgba="0.05 0.08 0.15 1.0"/>
+  </material>
   <!-- Base footprint on ground -->
   <link name="base_footprint"/>
@@ -8,5 +24,5 @@
     <child link="base_link"/>
   </joint>
-  <!-- JetTank Main Chassis Body -->
+  <!-- JetTank Main Chassis Body (Iconic Anodized Emerald Green Aluminum) -->
   <link name="base_link">
     <inertial>
@@ -18,28 +34,129 @@
       <origin xyz="0 0 0.04" rpy="0 0 0"/>
       <geometry>
-        <box size="0.26 0.20 0.10"/>
+        <box size="0.22 0.16 0.08"/>
       </geometry>
     </collision>
-    <visual>
-      <origin xyz="0 0 0.04" rpy="0 0 0"/>
-      <geometry>
-        <box size="0.26 0.20 0.10"/>
-      </geometry>
-      <material name="dark_gray">
-        <color rgba="0.2 0.22 0.25 1.0"/>
-      </material>
-    </visual>
-    <!-- Visual green accent stripe for JetTank -->
-    <visual>
-      <origin xyz="0.08 0 0.095" rpy="0 0 0"/>
-      <geometry>
-        <box size="0.08 0.16 0.01"/>
-      </geometry>
-      <material name="hiwonder_green">
-        <color rgba="0.1 0.75 0.3 1.0"/>
-      </material>
+    <!-- Visual 1: Main emerald green chassis hull -->
+    <visual>
+      <origin xyz="0 0 0.03" rpy="0 0 0"/>
+      <geometry>
+        <box size="0.18 0.16 0.06"/>
+      </geometry>
+      <material name="hiwonder_green"/>
+    </visual>
+    <!-- Visual 2: Sloped front nose plate -->
+    <visual>
+      <origin xyz="0.11 0 0.04" rpy="0 0.40 0"/>
+      <geometry>
+        <box size="0.08 0.16 0.006"/>
+      </geometry>
+      <material name="hiwonder_green"/>
+    </visual>
+    <!-- Visual 3: Front lower black bumper -->
+    <visual>
+      <origin xyz="0.115 0 0.015" rpy="0 0 0"/>
+      <geometry>
+        <box size="0.04 0.15 0.035"/>
+      </geometry>
+      <material name="jet_black"/>
+    </visual>
+    <!-- Visual 4: Front nose ventilation grill slot detail -->
+    <visual>
+      <origin xyz="0.135 0 0.04" rpy="0 0.40 0"/>
+      <geometry>
+        <box size="0.005 0.12 0.015"/>
+      </geometry>
+      <material name="jet_black"/>
+    </visual>
+    <!-- Visual 5: Middle green deck holding RPLiDAR -->
+    <visual>
+      <origin xyz="0.01 0 0.08" rpy="0 0 0"/>
+      <geometry>
+        <box size="0.14 0.15 0.005"/>
+      </geometry>
+      <material name="hiwonder_green"/>
+    </visual>
+    <!-- Visual 6: RPLiDAR lower base mount tray -->
+    <visual>
+      <origin xyz="0 0 0.095" rpy="0 0 0"/>
+      <geometry>
+        <cylinder radius="0.042" length="0.015"/>
+      </geometry>
+      <material name="jet_black"/>
+    </visual>
+    <!-- Visual 7: Upper green shelf bracket over RPLiDAR -->
+    <visual>
+      <origin xyz="0.01 0 0.14" rpy="0 0 0"/>
+      <geometry>
+        <box size="0.11 0.14 0.005"/>
+      </geometry>
+      <material name="hiwonder_green"/>
+    </visual>
+    <!-- Visual 8: Depth camera pan-tilt gimbal pedestal -->
+    <visual>
+      <origin xyz="0.02 0 0.155" rpy="0 0 0"/>
+      <geometry>
+        <cylinder radius="0.025" length="0.02"/>
+      </geometry>
+      <material name="jet_black"/>
+    </visual>
+    <!-- Visual 9: Depth camera sensor housing bar -->
+    <visual>
+      <origin xyz="0.03 0 0.185" rpy="0 0 0"/>
+      <geometry>
+        <box size="0.035 0.165 0.032"/>
+      </geometry>
+      <material name="jet_black"/>
+    </visual>
+    <!-- Visual 10: Depth camera optical lenses (Center RGB) -->
+    <visual>
+      <origin xyz="0.048 0 0.185" rpy="0 1.5707963 0"/>
+      <geometry>
+        <cylinder radius="0.009" length="0.005"/>
+      </geometry>
+      <material name="lens_glass"/>
+    </visual>
+    <!-- Visual 11: Depth camera optical lenses (Left IR) -->
+    <visual>
+      <origin xyz="0.048 0.045 0.185" rpy="0 1.5707963 0"/>
+      <geometry>
+        <cylinder radius="0.007" length="0.005"/>
+      </geometry>
+      <material name="lens_glass"/>
+    </visual>
+    <!-- Visual 12: Depth camera optical lenses (Right IR) -->
+    <visual>
+      <origin xyz="0.048 -0.045 0.185" rpy="0 1.5707963 0"/>
+      <geometry>
+        <cylinder radius="0.007" length="0.005"/>
+      </geometry>
+      <material name="lens_glass"/>
+    </visual>
+    <!-- Visual 13: Rear Jetson Nano & Display angled backplate -->
+    <visual>
+      <origin xyz="-0.08 0 0.11" rpy="0 -0.52 0"/>
+      <geometry>
+        <box size="0.10 0.14 0.05"/>
+      </geometry>
+      <material name="jet_black"/>
+    </visual>
+    <!-- Visual 14: Left Wi-Fi antenna -->
+    <visual>
+      <origin xyz="-0.08 0.055 0.18" rpy="0.20 -0.30 0"/>
+      <geometry>
+        <cylinder radius="0.004" length="0.10"/>
+      </geometry>
+      <material name="jet_black"/>
+    </visual>
+    <!-- Visual 15: Right Wi-Fi antenna -->
+    <visual>
+      <origin xyz="-0.08 -0.055 0.18" rpy="-0.20 -0.30 0"/>
+      <geometry>
+        <cylinder radius="0.004" length="0.10"/>
+      </geometry>
+      <material name="jet_black"/>
     </visual>
   </link>
-  <!-- Left Caterpillar Track Assembly (Dải bánh xích xe tăng bên trái) -->
+  <!-- Left Caterpillar Track Assembly (Dải bánh xích bên trái) -->
   <link name="left_wheel">
     <inertial>
@@ -48,5 +165,4 @@
       <inertia ixx="0.001" ixy="0" ixz="0" iyy="0.003" iyz="0" izz="0.003"/>
     </inertial>
-    <!-- Collision: main driving track base for skid-steer friction -->
     <collision>
       <origin xyz="0 0 0" rpy="1.5707963 0 0"/>
@@ -55,63 +171,136 @@
       </geometry>
     </collision>
-    <!-- Visual 1: Main continuous black rubber caterpillar track belt -->
-    <visual>
-      <origin xyz="0 0 0" rpy="0 0 0"/>
-      <geometry>
-        <box size="0.25 0.045 0.07"/>
-      </geometry>
-      <material name="track_rubber">
-        <color rgba="0.1 0.1 0.1 1.0"/>
-      </material>
-    </visual>
-    <!-- Visual 2: Front driving sprocket wheel -->
-    <visual>
-      <origin xyz="0.095 0 0" rpy="1.5707963 0 0"/>
-      <geometry>
-        <cylinder radius="0.035" length="0.047"/>
-      </geometry>
-      <material name="track_wheel">
-        <color rgba="0.25 0.28 0.32 1.0"/>
-      </material>
-    </visual>
-    <!-- Visual 3: Rear idler sprocket wheel -->
-    <visual>
-      <origin xyz="-0.095 0 0" rpy="1.5707963 0 0"/>
-      <geometry>
-        <cylinder radius="0.035" length="0.047"/>
-      </geometry>
-      <material name="track_wheel">
-        <color rgba="0.25 0.28 0.32 1.0"/>
-      </material>
-    </visual>
-    <!-- Visual 4: Middle road wheel 1 -->
-    <visual>
-      <origin xyz="-0.032 0 -0.005" rpy="1.5707963 0 0"/>
-      <geometry>
-        <cylinder radius="0.030" length="0.047"/>
-      </geometry>
-      <material name="track_wheel">
-        <color rgba="0.35 0.38 0.42 1.0"/>
-      </material>
-    </visual>
-    <!-- Visual 5: Middle road wheel 2 -->
-    <visual>
-      <origin xyz="0.032 0 -0.005" rpy="1.5707963 0 0"/>
-      <geometry>
-        <cylinder radius="0.030" length="0.047"/>
-      </geometry>
-      <material name="track_wheel">
-        <color rgba="0.35 0.38 0.42 1.0"/>
-      </material>
-    </visual>
-    <!-- Visual 6: Track top mudguard / fender -->
-    <visual>
-      <origin xyz="0 0 0.04" rpy="0 0 0"/>
-      <geometry>
-        <box size="0.26 0.05 0.008"/>
-      </geometry>
-      <material name="dark_gray">
-        <color rgba="0.2 0.22 0.25 1.0"/>
-      </material>
+    <!-- Visual 1: Outer metallic green sideplate with diagonal cutouts -->
+    <visual>
+      <origin xyz="0 0.024 0.005" rpy="0 0 0"/>
+      <geometry>
+        <box size="0.23 0.004 0.05"/>
+      </geometry>
+      <material name="hiwonder_green"/>
+    </visual>
+    <!-- Visual 2: Rear drive sprocket wheel (Green with holes) -->
+    <visual>
+      <origin xyz="-0.095 0 0.015" rpy="1.5707963 0 0"/>
+      <geometry>
+        <cylinder radius="0.038" length="0.044"/>
+      </geometry>
+      <material name="hiwonder_green"/>
+    </visual>
+    <!-- Visual 3: Rear sprocket silver hub -->
+    <visual>
+      <origin xyz="-0.095 0 0.015" rpy="1.5707963 0 0"/>
+      <geometry>
+        <cylinder radius="0.016" length="0.046"/>
+      </geometry>
+      <material name="metal_silver"/>
+    </visual>
+    <!-- Visual 4: Front raised idler wheel (Ramp climbing angle) -->
+    <visual>
+      <origin xyz="0.095 0 0.022" rpy="1.5707963 0 0"/>
+      <geometry>
+        <cylinder radius="0.035" length="0.044"/>
+      </geometry>
+      <material name="jet_black"/>
+    </visual>
+    <!-- Visual 5: Front idler silver hub -->
+    <visual>
+      <origin xyz="0.095 0 0.022" rpy="1.5707963 0 0"/>
+      <geometry>
+        <cylinder radius="0.012" length="0.046"/>
+      </geometry>
+      <material name="metal_silver"/>
+    </visual>
+    <!-- Visual 6: Bottom road wheel 1 -->
+    <visual>
+      <origin xyz="-0.045 0 -0.016" rpy="1.5707963 0 0"/>
+      <geometry>
+        <cylinder radius="0.027" length="0.044"/>
+      </geometry>
+      <material name="jet_black"/>
+    </visual>
+    <visual>
+      <origin xyz="-0.045 0 -0.016" rpy="1.5707963 0 0"/>
+      <geometry>
+        <cylinder radius="0.008" length="0.046"/>
+      </geometry>
+      <material name="metal_silver"/>
+    </visual>
+    <!-- Visual 7: Bottom road wheel 2 (Center) -->
+    <visual>
+      <origin xyz="0 0 -0.016" rpy="1.5707963 0 0"/>
+      <geometry>
+        <cylinder radius="0.027" length="0.044"/>
+      </geometry>
+      <material name="jet_black"/>
+    </visual>
+    <visual>
+      <origin xyz="0 0 -0.016" rpy="1.5707963 0 0"/>
+      <geometry>
+        <cylinder radius="0.008" length="0.046"/>
+      </geometry>
+      <material name="metal_silver"/>
+    </visual>
+    <!-- Visual 8: Bottom road wheel 3 -->
+    <visual>
+      <origin xyz="0.045 0 -0.016" rpy="1.5707963 0 0"/>
+      <geometry>
+        <cylinder radius="0.027" length="0.044"/>
+      </geometry>
+      <material name="jet_black"/>
+    </visual>
+    <visual>
+      <origin xyz="0.045 0 -0.016" rpy="1.5707963 0 0"/>
+      <geometry>
+        <cylinder radius="0.008" length="0.046"/>
+      </geometry>
+      <material name="metal_silver"/>
+    </visual>
+    <!-- Visual 9: Top return roller wheel -->
+    <visual>
+      <origin xyz="0 0 0.034" rpy="1.5707963 0 0"/>
+      <geometry>
+        <cylinder radius="0.018" length="0.044"/>
+      </geometry>
+      <material name="jet_black"/>
+    </visual>
+    <!-- Visual 10: Rubber caterpillar track belt - Bottom ground contact run -->
+    <visual>
+      <origin xyz="0 0 -0.041" rpy="0 0 0"/>
+      <geometry>
+        <box size="0.12 0.042 0.012"/>
+      </geometry>
+      <material name="matte_track"/>
+    </visual>
+    <!-- Visual 11: Rubber caterpillar track belt - Front upward ramp -->
+    <visual>
+      <origin xyz="0.09 0 -0.010" rpy="0 -0.55 0"/>
+      <geometry>
+        <box size="0.08 0.042 0.012"/>
+      </geometry>
+      <material name="matte_track"/>
+    </visual>
+    <!-- Visual 12: Rubber caterpillar track belt - Rear upward ramp -->
+    <visual>
+      <origin xyz="-0.09 0 -0.012" rpy="0 0.48 0"/>
+      <geometry>
+        <box size="0.08 0.042 0.012"/>
+      </geometry>
+      <material name="matte_track"/>
+    </visual>
+    <!-- Visual 13: Rubber caterpillar track belt - Top return run -->
+    <visual>
+      <origin xyz="0 0 0.050" rpy="0 0 0"/>
+      <geometry>
+        <box size="0.18 0.042 0.012"/>
+      </geometry>
+      <material name="matte_track"/>
+    </visual>
+    <!-- Visual 14: Top fender / mudguard -->
+    <visual>
+      <origin xyz="0 0 0.056" rpy="0 0 0"/>
+      <geometry>
+        <box size="0.24 0.048 0.005"/>
+      </geometry>
+      <material name="jet_black"/>
     </visual>
   </link>
@@ -122,5 +311,5 @@
     <axis xyz="0 1 0"/>
   </joint>
-  <!-- Right Caterpillar Track Assembly (Dải bánh xích xe tăng bên phải) -->
+  <!-- Right Caterpillar Track Assembly (Dải bánh xích bên phải) -->
   <link name="right_wheel">
     <inertial>
@@ -129,5 +318,4 @@
       <inertia ixx="0.001" ixy="0" ixz="0" iyy="0.003" iyz="0" izz="0.003"/>
     </inertial>
-    <!-- Collision: main driving track base for skid-steer friction -->
     <collision>
       <origin xyz="0 0 0" rpy="1.5707963 0 0"/>
@@ -136,63 +324,136 @@
       </geometry>
     </collision>
-    <!-- Visual 1: Main continuous black rubber caterpillar track belt -->
-    <visual>
-      <origin xyz="0 0 0" rpy="0 0 0"/>
-      <geometry>
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