Commit message: fix(simulation-stability): fix seesaw pitch with 4 base skids, enhance obstacle occlusion, suppress EOL popup, and refine scientific paper visuals

File: 04_demo_simulation/ros1/mars_online_jettank/urdf/jettank.urdf.xacro (robot description, xacro)
@@ -28,6 +28,6 @@
     <inertial>
       <mass value="2.5"/>
-      <origin xyz="0 0 0.04" rpy="0 0 0"/>
-      <inertia ixx="0.015" ixy="0" ixz="0" iyy="0.020" iyz="0" izz="0.025"/>
+      <origin xyz="0 0 0.01" rpy="0 0 0"/>
+      <inertia ixx="0.02" ixy="0" ixz="0" iyy="0.03" iyz="0" izz="0.03"/>
     </inertial>
     <collision>
@@ -35,4 +35,29 @@
       <geometry>
         <box size="0.22 0.16 0.08"/>
+      </geometry>
+    </collision>
+    <!-- 4 Non-rotating anti-pitch/anti-tip track skids in base_link (front/rear of each track) -->
+    <collision name="left_track_front_skid">
+      <origin xyz="0.08 0.11 -0.001" rpy="0 0 0"/>
+      <geometry>
+        <sphere radius="0.044"/>
+      </geometry>
+    </collision>
+    <collision name="left_track_rear_skid">
+      <origin xyz="-0.08 0.11 -0.001" rpy="0 0 0"/>
+      <geometry>
+        <sphere radius="0.044"/>
+      </geometry>
+    </collision>
+    <collision name="right_track_front_skid">
+      <origin xyz="0.08 -0.11 -0.001" rpy="0 0 0"/>
+      <geometry>
+        <sphere radius="0.044"/>
+      </geometry>
+    </collision>
+    <collision name="right_track_rear_skid">
+      <origin xyz="-0.08 -0.11 -0.001" rpy="0 0 0"/>
+      <geometry>
+        <sphere radius="0.044"/>
       </geometry>
     </collision>
@@ -165,4 +190,5 @@
       <inertia ixx="0.001" ixy="0" ixz="0" iyy="0.003" iyz="0" izz="0.003"/>
     </inertial>
+    <!-- Continuous concentric driving cylinder (ground contact with high track traction) -->
     <collision>
       <origin xyz="0 0 0" rpy="1.5707963 0 0"/>
@@ -318,4 +344,5 @@
       <inertia ixx="0.001" ixy="0" ixz="0" iyy="0.003" iyz="0" izz="0.003"/>
     </inertial>
+    <!-- Continuous concentric driving cylinder (ground contact with high track traction) -->
     <collision>
       <origin xyz="0 0 0" rpy="1.5707963 0 0"/>
@@ -471,10 +498,4 @@
       <inertia ixx="0.0001" ixy="0" ixz="0" iyy="0.0001" iyz="0" izz="0.0001"/>
     </inertial>
-    <collision>
-      <origin xyz="0 0 0" rpy="0 0 0"/>
-      <geometry>
-        <cylinder radius="0.036" length="0.035"/>
-      </geometry>
-    </collision>
     <!-- RPLiDAR black rotating cylindrical turret -->
     <visual>
@@ -501,4 +522,6 @@
   <!-- Gazebo Material Colors -->
   <gazebo reference="base_link">
+    <mu1>0.05</mu1>
+    <mu2>0.05</mu2>
     <material>Gazebo/Green</material>
   </gazebo>
